File: Circuit Boards/BackPlane/BackPlane.kicad_pcb (KiCad board)
At the start: 4 copper layers, 390 x 128 mm, 72 parts, among them J1 DIN41612-C-96-F, J10 DIN41612-C-96-F, J11 DIN41612-C-96-F, J12 DIN41612-C-96-F, J13 DIN41612-C-96-F, J14 DIN41612-C-96-F, J15 DIN41612-C-96-F, J16 DIN41612-C-96-F, J17 4771 3-pin, J18 DIN41612-H-15-F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

Commit message: Backplane: Initial PCB layout
Parts:
- moved MH1 0.51 mm to (22.6, 89.4)
Routing:
- net VTT: track 0.00 -> 1736.8 mm
- net +3V3: track 0.00 -> 1544.5 mm
- net +5V: track 0.00 -> 1482.3 mm
- net GND: track 0.00 -> 1120.1 mm
- net D15: track 0.00 -> 367.5 mm
- net A24: track 0.00 -> 367.5 mm
- net A21: track 0.00 -> 367.5 mm
- net A17: track 0.00 -> 367.5 mm
- net A15: track 0.00 -> 367.5 mm
- net A11: track 0.00 -> 367.5 mm
- net A08: track 0.00 -> 367.5 mm
- net STERM: track 0.00 -> 367.5 mm
- net SIZ1: track 0.00 -> 367.5 mm
- net IRQ5: track 0.00 -> 367.5 mm
- net IRQ1: track 0.00 -> 367.5 mm
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- added copper zone on B.Cu, net GND
- added copper zone on F.Cu, net GND
- added copper zone on In1.Cu, net GND
- added copper zone on In2.Cu, net GND
Other:
- board text added: "Inner 1 Copper"
- board text added: "Inner 2 Copper"
